File: CAD/KiCad/AVA/_autosave-AVA.kicad_sch (KiCad schematic)
At the start: 3 parts, among them J1 Conn_01x40_Pin, M1 Motor_Servo

Commit message: Working on schematic.
Other:
- moved on the sheet: U1
Changed lines of the file:
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@@
 	(symbol
 		(lib_id "AVA:ESC_Servo")
-		(at 168.91 72.39 0)
+		(at 168.91 38.1 0)
 		(unit 1)
 		(body_style 1)
@@
 		(fields_autoplaced yes)
 		(property "Reference" "U1"
-			(at 175.26 71.12 0)
+			(at 175.26 36.83 0)
 			(show_name no)
 			(do_not_autoplace no)
@@
 		)
 		(property "Value" ""
-			(at 168.91 72.39 0)
+			(at 168.91 38.1 0)
 			(show_name no)
 			(do_not_autoplace no)
@@
 		)
 		(property "Footprint" ""
-			(at 168.91 72.39 0)
+			(at 168.91 38.1 0)
 			(hide yes)
 			(show_name no)
@@
 		)
 		(property "Datasheet" ""
-			(at 168.91 72.39 0)
+			(at 168.91 38.1 0)
 			(hide yes)
 			(show_name no)
@@
 		)
 		(property "Description" ""
-			(at 168.91 72.39 0)
+			(at 168.91 38.1 0)
 			(hide yes)
 			(show_name no)
