File: CAD/KiCad/AVA/AVA.kicad_sch (KiCad schematic)
At the start: 3 parts, among them J1 Conn_01x40_Pin, M1 Motor_Servo

Commit message: Absolutely barebones, borderline starving schematic done. Probably fucked up, earned ciggie break tho
Parts:
- added C2: C_Polarized_US, symbol Device:C_Polarized_US
- added J2: Barrel_Jack, Connector_BarrelJack:BarrelJack_SwitchcraftConxall_RAPC10U_Horizontal, symbol Connector:Barrel_Jack
- added M2: Steering_Front_Servo, Connector_PinHeader_2.54mm:PinHeader_1x03_P2.54mm_Vertical, symbol Motor:Motor_Servo
- added M3: Steering_Back_Servo, Connector_PinHeader_2.54mm:PinHeader_1x03_P2.54mm_Vertical, symbol Motor:Motor_Servo
- added M4: Fan, symbol Motor:Fan
- added SW1: SW_Push, symbol Switch:SW_Push
Connections:
- net 5.0VDC is gone; now on net +5V: J1.2 (Pin_2), J1.4 (Pin_4)
- net GND: now also U1.7 (GND_{uC}), U1.8 (GND_{T-Conn}), J2.2, M2.3 (-), M3.3 (-)
- net GPIO-12: now also M2.1 (PWM)
- net GPIO01: now also M3.1 (PWM)
- net GPIO09: now also U1.6 (PWM_{uC})
- net at M1.1 (PWM): now also U1.3 (PWM_{Servo})
- net at M1.2 (+): now also U1.2 (VCC_{Servo})
- net at M1.3 (-): now also U1.4 (GND_{Servo})
- net BMU/U_{Bat1+Bat2-Unregulated}: now reaches U1.1 (VCC_{T-Conn})
- net at U1.10 (VCC_{Ripple}): now also C2.1
- net at U1.11 (GND): now also M4.2 (-)
- net at U1.12 (Fan): now also M4.1 (+)
- net at U1.13 (VCC): now also SW1.2
- net at U1.14 (~{EN}): now also SW1.1
- net +5V: now reaches U1.5 (VCC_{uC})
- net +5V: now also M2.2 (+), M3.2 (+)
- net at U1.9 (GND_{Ripple}): now also C2.2
- net 3.3VDC renamed +3.3V
- new net BMU/U_{Bat-Regulated}: J2.1
Other:
- sheet BMU ports: added U_{Bat-Regulated}, U_{Bat1+Bat2-Unregulated}; removed 5V, VCC
- moved on the sheet: J1, M1, U1
