File: CAD/KiCad/AVA/AVA.kicad_sch (KiCad schematic)
At the start: 48 parts, among them J1 Conn_01x03_Pin, J10 Conn_01x04_Pin, J2 Conn_01x03_Pin, J3 Conn_01x03_Pin, J4 Conn_01x03_Pin, J5 Conn_01x02_Pin, J6 Conn_01x02_Pin, J7 Conn_01x02_Pin, J8 Conn_01x03_Pin, J9 Conn_01x03_Pin, U1 ESP32-C3-Super-Mini, U2 ESP32-DevKitC

Commit message: Digital hall wire, using GPIO2/8/9 from ESP32-C3-SuperMini not necessary. Changed to digital only GPIO
Connections:
- net at R8.2: now also U1.3 (SS/GPIO7); no longer U1.12 (A3/GPIO3)
- net at R10.2: now also U1.6 (GPIO10); no longer U1.13 (SCLK/A4/GPIO4)
- net at U1.11 (A2/GPIO2): no longer R6.2
- net at U1.2 (POSI/GPIO6): now also R6.2
Changed lines of the file:
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@@
-	(wire
-		(pts
-			(xy 152.4 59.69) (xy 152.4 77.47)
-		)
-		(stroke
-			(width 0)
-			(type default)
-		)
-	)
 	(wire
 		(pts
@@
 	(wire
 		(pts
-			(xy 152.4 77.47) (xy 102.87 77.47)
-		)
-		(stroke
-			(width 0)
-			(type default)
-		)
-	)
-	(wire
-		(pts
 			(xy 151.13 74.93) (xy 151.13 62.23)
 		)
@@
 	(wire
 		(pts
-			(xy 93.98 43.18) (xy 102.87 43.18)
+			(xy 93.98 43.18) (xy 97.79 43.18)
 		)
 		(stroke
@@
 	(wire
 		(pts
-			(xy 148.59 57.15) (xy 153.67 57.15)
-		)
-		(stroke
-			(width 0)
-			(type default)
-		)
-	)
-	(wire
-		(pts
 			(xy 53.34 71.12) (xy 85.09 71.12)
 		)
@@
 	(wire
 		(pts
+			(xy 109.22 52.07) (xy 99.06 52.07)
+		)
+		(stroke
+			(width 0)
+			(type default)
+		)
+	)
+	(wire
+		(pts
 			(xy 49.53 182.88) (xy 76.2 182.88)
 		)
@@
 	(wire
 		(pts
-			(xy 102.87 77.47) (xy 102.87 57.15)
-		)
-		(stroke
-			(width 0)
-			(type default)
-		)
-	)
-	(wire
-		(pts
-			(xy 109.22 46.99) (xy 102.87 46.99)
+			(xy 109.22 46.99) (xy 97.79 46.99)
 		)
 		(stroke
@@
 	(wire
 		(pts
+			(xy 97.79 49.53) (xy 97.79 57.15)
+		)
+		(stroke
+			(width 0)
+			(type default)
+		)
+	)
+	(wire
+		(pts
 			(xy 62.23 74.93) (xy 64.77 74.93)
 		)
@@
 	(wire
 		(pts
+			(xy 109.22 49.53) (xy 97.79 49.53)
+		)
+		(stroke
+			(width 0)
+			(type default)
+		)
+	)
+	(wire
+		(pts
 			(xy 93.98 86.36) (xy 101.6 86.36)
 		)
@@
 	(wire
 		(pts
+			(xy 109.22 59.69) (xy 101.6 59.69)
+		)
+		(stroke
+			(width 0)
+			(type default)
+		)
+	)
+	(wire
+		(pts
 			(xy 127 177.8) (xy 138.43 177.8)
 		)
@@
 	(wire
 		(pts
-			(xy 153.67 78.74) (xy 101.6 78.74)
-		)
-		(stroke
-			(width 0)
-			(type default)
-		)
-	)
-	(wire
-		(pts
 			(xy 124.46 114.3) (xy 162.56 114.3)
 		)
@@
 	(wire
 		(pts
+			(xy 99.06 52.07) (xy 99.06 71.12)
+		)
+		(stroke
+			(width 0)
+			(type default)
+		)
+	)
+	(wire
+		(pts
 			(xy 187.96 102.87) (xy 186.69 102.87)
 		)
@@
 	(wire
 		(pts
-			(xy 148.59 59.69) (xy 152.4 59.69)
-		)
-		(stroke
-			(width 0)
-			(type default)
-		)
-	)
-	(wire
-		(pts
 			(xy 166.37 60.96) (xy 190.5 60.96)
 		)
@@
 	(wire
 		(pts
-			(xy 101.6 80.01) (xy 154.94 80.01)
-		)
-		(stroke
-			(width 0)
-			(type default)
-		)
-	)
-	(wire
-		(pts
 			(xy 186.69 105.41) (xy 186.69 102.87)
 		)
@@
 	(wire
 		(pts
-			(xy 102.87 57.15) (xy 93.98 57.15)
-		)
-		(stroke
-			(width 0)
-			(type default)
-		)
-	)
-	(wire
-		(pts
 			(xy 147.32 179.07) (xy 147.32 177.8)
 		)
@@
 	(wire
 		(pts
-			(xy 102.87 46.99) (xy 102.87 43.18)
+			(xy 97.79 43.18) (xy 97.79 46.99)
 		)
 		(stroke
@@
 	(wire
 		(pts
-			(xy 148.59 54.61) (xy 154.94 54.61)
-		)
-		(stroke
-			(width 0)
-			(type default)
-		)
-	)
-	(wire
-		(pts
 			(xy 64.77 74.93) (xy 64.77 77.47)
 		)
@@
 	(wire
 		(pts
+			(xy 101.6 59.69) (xy 101.6 86.36)
+		)
+		(stroke
+			(width 0)
+			(type default)
+		)
+	)
+	(wire
+		(pts
 			(xy 121.92 180.34) (xy 128.27 180.34)
 		)
@@
 	(wire
 		(pts
-			(xy 101.6 86.36) (xy 101.6 80.01)
-		)
-		(stroke
-			(width 0)
-			(type default)
-		)
-	)
-	(wire
-		(pts
 			(xy 54.61 74.93) (xy 40.64 74.93)
 		)
@@
 	(wire
 		(pts
+			(xy 97.79 57.15) (xy 93.98 57.15)
+		)
+		(stroke
+			(width 0)
+			(type default)
+		)
+	)
+	(wire
+		(pts
 			(xy 85.09 62.23) (xy 74.93 62.23)
 		)
@@
 	(wire
 		(pts
-			(xy 153.67 57.15) (xy 153.67 78.74)
-		)
-		(stroke
-			(width 0)
-			(type default)
-		)
-	)
-	(wire
-		(pts
 			(xy 74.93 48.26) (xy 74.93 34.29)
 		)
@@
 	(wire
 		(pts
-			(xy 101.6 78.74) (xy 101.6 71.12)
-		)
-		(stroke
-			(width 0)
-			(type default)
-		)
-	)
-	(wire
-		(pts
 			(xy 49.53 166.37) (xy 80.01 166.37)
 		)
@@
 	(wire
 		(pts
-			(xy 93.98 71.12) (xy 101.6 71.12)
+			(xy 93.98 71.12) (xy 99.06 71.12)
 		)
 		(stroke
@@
 		)
 		(stroke
-			(width 0)
-			(type default)
-		)
-	)
-	(wire
-		(pts
-			(xy 154.94 54.61) (xy 154.94 80.01)
-		)
-		(stroke
