File: CAD/KiCad/AVA/BMU.kicad_sch (KiCad schematic)
At the start: 8 parts, among them Q1 IRF9540N

Commit message: Absolutely barebones, borderline starving schematic done. Probably fucked up, earned ciggie break tho
Parts:
- added D2: MBR745, Package_TO_SOT_THT:TO-220-2_Vertical, symbol Diode:MBR745
- D1: value 5V -> 6.2V
Connections:
- net 5V: no longer names the net of D1.1 (K), Q1.3 (S)
- net 5V: now also D2.2 (A); no longer C1.1
- net VCC renamed U_{Bat1+Bat2-Unregulated}
- new net U_{Bat-Regulated}: C1.1, D2.1 (K)
Other:
- moved on the sheet: BT1, BT2, BT3, BT4, C1, D1, Q1, R1
