File: CAD/KiCad/AVA/_autosave-AVA.kicad_pcb (KiCad board)
At the start: 2 copper layers, 100 x 75 mm, 48 parts, among them J1 Conn_01x03_Pin, J10 Conn_01x04_Pin, J2 Conn_01x03_Pin, J3 Conn_01x03_Pin, J4 Conn_01x03_Pin, J5 Conn_01x02_Pin, J6 Conn_01x02_Pin, J7 Conn_01x02_Pin, J8 Conn_01x03_Pin, J9 Conn_01x03_Pin, U1 WEMOS_C3_mini

Commit message: 50% of layout done. We buried them wrong
Parts:
- moved J10 106.0 mm to (164.3, 86.7)
- moved J8 106.0 mm to (174.5, 69.8)
- moved J9 106.0 mm to (179.1, 69.8)
- moved J5 106.0 mm to (164.3, 79.5)
Routing:
- net Net-(U1-3V3): track 0.00 -> 45.7 mm, vias 0 -> 4
Changed lines of the file:
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@@
 	(footprint "Connector_PinSocket_2.54mm:PinSocket_1x04_P2.54mm_Vertical"
 		(layer "F.Cu")
-		(at 138.87 189.52)
+		(at 164.27 86.65)
 		(descr "Through hole straight socket strip, 1x04, 2.54mm pitch, single row (from Kicad 4.0.7), script generated")
 		(tags "Through hole socket strip THT 1x04 2.54mm single row")
@@
 	(footprint "Connector_PinSocket_2.54mm:PinSocket_1x03_P2.54mm_Vertical"
 		(layer "F.Cu")
-		(at 153.67 172.72)
+		(at 179.07 69.85)
 		(descr "Through hole straight socket strip, 1x03, 2.54mm pitch, single row (from Kicad 4.0.7), script generated")
 		(tags "Through hole socket strip THT 1x03 2.54mm single row")
@@
 	(footprint "Connector_PinSocket_2.54mm:PinSocket_1x03_P2.54mm_Vertical"
 		(layer "F.Cu")
-		(at 149.08 172.72)
+		(at 174.48 69.85)
 		(descr "Through hole straight socket strip, 1x03, 2.54mm pitch, single row (from Kicad 4.0.7), script generated")
 		(tags "Through hole socket strip THT 1x03 2.54mm single row")
@@
 	(footprint "Connector_PinSocket_2.54mm:PinSocket_1x02_P2.54mm_Vertical"
 		(layer "F.Cu")
-		(at 138.87 182.39)
+		(at 164.27 79.52)
 		(descr "Through hole straight socket strip, 1x02, 2.54mm pitch, single row (from Kicad 4.0.7), script generated")
 		(tags "Through hole socket strip THT 1x02 2.54mm single row")
@@
 	)
 	(segment
+		(start 161.29 72.39)
+		(end 161.29 62.23)
+		(width 0.8)
+		(layer "F.Cu")
+		(net "Net-(U1-3V3)")
+	)
+	(segment
+		(start 161.29 82.55)
+		(end 161.29 72.39)
+		(width 0.8)
+		(layer "F.Cu")
+		(net "Net-(U1-3V3)")
+	)
+	(segment
+		(start 161.29 92.71)
+		(end 161.29 82.55)
+		(width 0.8)
+		(layer "F.Cu")
+		(net "Net-(U1-3V3)")
+	)
+	(via
+		(at 161.29 92.71)
+		(size 1.6)
+		(drill 0.8)
+		(layers "F.Cu" "B.Cu")
+		(net "Net-(U1-3V3)")
+	)
+	(via
+		(at 161.29 62.23)
+		(size 1.6)
+		(drill 0.8)
+		(layers "F.Cu" "B.Cu")
+		(net "Net-(U1-3V3)")
+	)
+	(via
+		(at 161.29 72.39)
+		(size 1.6)
+		(drill 0.8)
+		(layers "F.Cu" "B.Cu")
+		(net "Net-(U1-3V3)")
+	)
+	(via
+		(at 161.29 82.55)
+		(size 1.6)
+		(drill 0.8)
+		(layers "F.Cu" "B.Cu")
+		(net "Net-(U1-3V3)")
+	)
+	(segment
+		(start 157.48 82.55)
+		(end 161.29 82.55)
+		(width 0.8)
+		(layer "B.Cu")
+		(net "Net-(U1-3V3)")
+	)
+	(segment
+		(start 157.48 72.39)
+		(end 161.29 72.39)
+		(width 0.8)
+		(layer "B.Cu")
+		(net "Net-(U1-3V3)")
+	)
+	(segment
+		(start 157.48 92.71)
+		(end 161.29 92.71)
+		(width 0.8)
+		(layer "B.Cu")
+		(net "Net-(U1-3V3)")
+	)
+	(segment
+		(start 157.48 62.23)
+		(end 161.29 62.23)
+		(width 0.8)
+		(layer "B.Cu")
+		(net "Net-(U1-3V3)")
+	)
+	(segment

Commit message: 75% done. Signal integrity is a myth invented by Bosch to sell expensive cables
Parts:
- moved C6 143.4 mm to (179.7, 80.6)
- moved C5 137.3 mm to (179.7, 90.2)
- moved R11 127.9 mm to (177.2, 83.8)
- moved R12 127.3 mm to (177.2, 87.0)
- moved R14 126.6 mm to (177.2, 77.5)
- moved R13 126.4 mm to (177.2, 74.3)
- moved J6 119.5 mm to (173.4, 74.3)
- moved R18 77.8 mm to (190.5, 122.6), turned to 180 degrees
- moved J8 64.1 mm to (137.2, 121.9), turned to 90 degrees
- moved J9 58.5 mm to (152.4, 121.9), turned to 90 degrees
- moved R21 48.4 mm to (189.9, 94.3), turned to 180 degrees
- moved R26 47.1 mm to (158.8, 113.0), turned to 180 degrees
- moved J5 46.1 mm to (146.1, 121.9), turned to 90 degrees
- moved R20 42.8 mm to (189.9, 97.8), turned to 180 degrees
- moved R25 42.1 mm to (135.9, 113.0)
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Routing:
- net Net-(A1-D4): track 0.00 -> 101.3 mm
- net Net-(A1-D5): track 0.00 -> 97.5 mm
- net Net-(A1-D7): track 0.00 -> 59.4 mm
- net Net-(U1-3V3): track 45.7 -> 105.0 mm
- net Net-(A1-D6): track 0.00 -> 59.0 mm
- net Net-(A1-D3): track 2.54 -> 60.1 mm
- net Net-(A1-D2): track 2.69 -> 57.0 mm
- net /6.2V: track 0.00 -> 37.6 mm
- net Net-(U1-D2): track 0.00 -> 27.5 mm
- net Net-(U1-D3): track 0.00 -> 23.8 mm
- net Net-(A1-D1/TX): track 56.5 -> 78.0 mm
- net /CH2: track 0.00 -> 16.0 mm
- net /CH1: track 0.00 -> 12.5 mm
- net Net-(A1-D0/RX): track 54.4 -> 66.0 mm
- net Net-(U1-TX): track 35.4 -> 45.7 mm
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