File: CAD/KiCad/AVA/_autosave-AVA.kicad_pcb (KiCad board)
At the start: 2 copper layers, 100 x 75 mm, 48 parts, among them J1 Conn_01x03_Pin, J10 Conn_01x04_Pin, J2 Conn_01x03_Pin, J3 Conn_01x03_Pin, J4 Conn_01x03_Pin, J5 Conn_01x02_Pin, J6 Conn_01x02_Pin, J7 Conn_01x02_Pin, J8 Conn_01x03_Pin, J9 Conn_01x03_Pin

Commit message: Back, front finished. Cropped svg for printing, 500 cigarettes
Routing:
- net GND: vias 6 -> 8
Changed lines of the file:
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@@
 			(outputformat 5)
 			(mirror no)
-			(drillshape 0)
+			(drillshape 2)
 			(scaleselection 1)
 			(outputdirectory "FAB/SVG/")
@@
 	)
 	(segment
+		(start 163.83 94.615)
+		(end 163.83 104.565)
+		(width 0.8)
+		(layer "F.Cu")
+		(net "GND")
+	)
+	(segment
 		(start 163.83 70.485)
 		(end 163.83 62.23)
@@
 	(segment
 		(start 163.83 84.455)
-		(end 163.83 104.565)
+		(end 163.83 92.71)
 		(width 0.8)
 		(layer "F.Cu")
@@
 		(net "GND")
 	)
+	(segment
+		(start 163.83 92.71)
+		(end 163.83 94.615)
+		(width 0.8)
+		(layer "F.Cu")
+		(net "GND")
+	)
 	(via
 		(at 163.83 104.565)
@@
 	)
 	(via
+		(at 163.83 92.71)
+		(size 1.6)
+		(drill 0.8)
+		(layers "F.Cu" "B.Cu")
+		(net "GND")
+	)
+	(via
 		(at 163.83 70.485)
 		(size 1.6)
@@
 		(net "GND")
 	)
+	(via
+		(at 163.83 94.615)
+		(size 1.6)
+		(drill 0.8)
+		(layers "F.Cu" "B.Cu")
+		(net "GND")
+	)

Commit message: Track width min now 1.6mm. Double sided board, no pre-drawn holes in front, back svg for easy printing
Parts:
- moved R1 49.0 mm to (177.2, 103.5)
- moved R2 49.0 mm to (173.4, 103.5)
- moved R21 33.7 mm to (208.3, 122.6), turned to 0 degrees
- moved R20 28.4 mm to (208.3, 119.4), turned to 0 degrees
- moved R18 8.25 mm to (182.2, 122.6)
- moved R19 8.25 mm to (172.1, 119.4)
Connections:
- net Net-(J1-Pin_1) renamed VCC
Routing:
- net VCC: track 214.3 -> 0.00 mm
- net Net-(A1-D1/TX): track 79.5 -> 10.6 mm
- net Net-(U1-D0): track 127.5 -> 63.3 mm, vias 0 -> 2
- net Net-(A1-D0/RX): track 65.7 -> 10.4 mm
- net Net-(U1-D1): track 123.6 -> 68.6 mm, vias 0 -> 2
- net Net-(U1-3.3V): track 138.7 -> 89.9 mm, vias 6 -> 1
- net Net-(U1-TX): track 49.1 -> 97.5 mm
- net Net-(U1-RX): track 51.6 -> 95.6 mm
- net GND: track 40.4 -> 0.00 mm, vias 8 -> 0
- net Net-(U1-D2): track 114.5 -> 81.7 mm, vias 0 -> 2
- net Net-(A1-D4): track 101.3 -> 82.6 mm, vias 0 -> 2
- net Net-(J7-Pin_2): track 5.61 -> 15.9 mm
- net Net-(A1-D7): track 59.4 -> 49.7 mm
- net /CH1: track 12.5 -> 4.23 mm
- net /CH2: track 16.0 -> 8.53 mm
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- added copper zone on F.Cu, net VCC

Commit message: ESP32-C3-SuperMini and Arduino Nano ESP32 layout. Next variant ESP32-C3-SuperMini and ESP32-WROOM-32U
Parts:
- U1: value ~ -> ESP32-C3-Super-Mini
- moved U1 0.53 mm to (204.4, 73.4), turned to 90 degrees
Connections:
- C5 pad 2: Net-(U1-D10) -> Net-(U1-A1/GPIO1)
- C6 pad 2: Net-(U1-D9) -> Net-(U1-A0/GPIO0)
- R1 pad 1: Net-(U1-RX) -> Net-(U1-TX/GPIO21)
- R10 pad 2: Net-(U1-D0) -> Net-(U1-GPIO10)
- R11 pad 2: Net-(U1-D10) -> Net-(U1-A1/GPIO1)
- R12 pad 2: Net-(U1-D10) -> Net-(U1-A1/GPIO1)
- R13 pad 2: Net-(U1-D9) -> Net-(U1-A0/GPIO0)
- R14 pad 2: Net-(U1-D9) -> Net-(U1-A0/GPIO0)
- R2 pad 1: Net-(U1-TX) -> Net-(U1-RX/GPIO20)
- R3 pad 2: Net-(U1-D3) -> Net-(U1-PISO/GPIO5)
- R6 pad 2: Net-(U1-D2) -> Net-(U1-POSI/GPIO6)
- R8 pad 2: Net-(U1-D1) -> Net-(U1-SS/GPIO7)
- U1 pad 1: unconnected-(U1-D5-Pad1) -> Net-(U1-PISO/GPIO5)
- U1 pad 10: Net-(U1-D1) -> Net-(U1-A1/GPIO1)
- U1 pad 11: Net-(U1-D2) -> unconnected-(U1-A2/GPIO2-Pad11)
- U1 pad 12: Net-(U1-D3) -> unconnected-(U1-A3/GPIO3-Pad12)
- U1 pad 2: unconnected-(U1-D6-Pad2) -> Net-(U1-POSI/GPIO6)
- U1 pad 3: unconnected-(U1-D7-Pad3) -> Net-(U1-SS/GPIO7)
- U1 pad 5: Net-(U1-D9) -> unconnected-(U1-SCLK/GPIO9-Pad5)
- U1 pad 6: Net-(U1-D10) -> Net-(U1-GPIO10)
- U1 pad 7: Net-(U1-RX) -> Net-(U1-RX/GPIO20)
- U1 pad 8: Net-(U1-TX) -> Net-(U1-TX/GPIO21)
- U1 pad 9: Net-(U1-D0) -> Net-(U1-A0/GPIO0)
Routing:
- net Net-(U1-GPIO10): track 0.00 -> 124.4 mm
- net Net-(U1-SS/GPIO7): track 0.00 -> 118.1 mm
- net Net-(U1-PISO/GPIO5): track 0.00 -> 114.2 mm
- net Net-(U1-POSI/GPIO6): track 0.00 -> 114.0 mm
- net Net-(U1-D3): track 107.9 -> 0.00 mm, vias 2 -> 0
- net Net-(U1-TX): track 97.5 -> 0.00 mm
- net Net-(U1-RX): track 95.6 -> 0.00 mm
- net Net-(U1-D2): track 81.7 -> 0.00 mm, vias 2 -> 0
- net Net-(U1-D1): track 68.6 -> 0.00 mm, vias 2 -> 0
- net Net-(U1-D0): track 63.3 -> 0.00 mm, vias 2 -> 0
- net Net-(U1-RX/GPIO20): track 0.00 -> 42.4 mm
- net Net-(U1-D10): track 38.8 -> 0.00 mm
- net Net-(U1-D9): track 35.8 -> 0.00 mm
- net Net-(U1-TX/GPIO21): track 0.00 -> 34.8 mm
- net Net-(U1-A1/GPIO1): track 0.00 -> 33.9 mm
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